File: pcb/finalMidiGuitar.kicad_sch (KiCad schematic)
At the start: 20 parts, among them J1 PinHeader_01x06_P2.54mm_Verti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, J3 NeoPixel, J4 Oled Display, M1 Module_XIAO_Generic_SocketSMD, SW1 BTN, U1 LevelShifter

Commit message: Refactor code structure for improved readability and maintainability
Parts:
- removed C4, C5: 0.1uf, PCM_fab:C_1206, symbol PCM_fab:C_1206
- removed D1: Diode_Schottky_MiniSMA, PCM_fab:Diode_Schottky_MiniSMA, symbol PCM_fab:Diode_Schottky_MiniSMA
- removed J1: PinHeader_01x06_P2.54mm_Vertical_THT_D1mm, PCM_fab:PinHeader_01x06_P2.54mm_Vertical_THT_D1mm, symbol PCM_fab:PinHeader_01x06_P2.54mm_Vertical_THT_D1mm
- removed R2, R3, R4: 10 kΩ, PCM_fab:R_1206, symbol PCM_fab:R_1206
- removed R5, R7, R8: 0, PCM_fab:R_1206, symbol PCM_fab:R_1206
- removed U1: LevelShifter, PCM_fab:LevelShifter_Texas_TXB0104DR_SOIC-14, symbol PCM_fab:LevelShifter_Texas_TXB0104DR_SOIC-14
- added J1: NeoPixel, PCM_fab:PinHeader_01x04_P2.54mm_Vertical_THT_D1mm, symbol PCM_fab:PinHeader_01x04_P2.54mm_Vertical_THT_D1mm
- added U1: SN74LVC1T45DBVR, DBV0006A_N, symbol 2026-04-11_16-51-34:SN74LVC1T45DBVR
Connections:
- net 4V5_NEO is gone; now on net PWR_5V: C3.2, J3.2 (Pin_2)
- net PWR_3V3: now also J1.3 (Pin_3), U1.1 (VCCA), U1.5 (DIR)
- net PWR_5V: now also U1.6 (VCCB)
- net PWR_GND: now also J1.4 (Pin_4), U1.2 (GND)
- net SCL: now also J1.1 (Pin_1)
- net SDA: now also J1.2 (Pin_2)
- net at R1.1: now also U1.4 (B)
- net at M1.11 (D10): now also U1.3 (A)
- net INT: no longer names the net of M1.1 (D0)
- net XSHUT: no longer names the net of M1.7 (D6)
- no-connect marks 5 -> 4
Other:
- moved on the sheet: C1
