File: finalMidiGuitar/finalMidiGuitar.kicad_pcb (KiCad board)
At the start: 2 copper layers, 68.1 x 30.3 mm, 51 parts, among them J1 NeoPixel, J3 NeoPixel, J4 Oled Display, M1 Module_XIAO_Generic_SocketSMD, SW1 BTN, U1 SN74LVC1T45DBVR

Commit message: Add label "Midi Guitar" to the schematic for better identification
Routing:
- net PWR_GND: track 24.1 -> 36.6 mm, vias 2 -> 0
- net PWR_5V: track 87.1 -> 90.4 mm
- net PWR_3V3: track 144.6 -> 147.7 mm
- net SCL: track 72.8 -> 75.6 mm
- net Net-(U1-B): track 3.36 -> 5.36 mm
- net Net-(M1-D10): track 61.7 -> 60.7 mm
- net Net-(M1-D3): track 34.6 -> 35.6 mm
- net SDA: track 71.3 -> 72.3 mm
- net Net-(J3-Pin_1): track 21.9 -> 21.0 mm
- net Net-(M1-D2): track 34.5 -> 34.1 mm, vias 2 -> 0

Commit message: Refactor code structure for improved readability and maintainability
Parts:
- moved J3 5.15 mm to (139.1, 120.2)
- moved ? 0.45 mm to (158.7, 134.4)
- moved ? 0.45 mm to (158.2, 134.4)
- moved REF** 0.45 mm to (158.7, 134.4)
- moved REF** 0.45 mm to (158.2, 134.4)
- moved ? 0.45 mm to (157.7, 134.4)
- moved REF** 0.45 mm to (157.7, 134.4)
- moved ? 0.45 mm to (158.7, 123.2)
- moved ? 0.45 mm to (158.2, 123.2)
- moved REF** 0.45 mm to (158.7, 123.2)
- moved REF** 0.45 mm to (158.2, 123.2)
- moved ? 0.45 mm to (157.7, 123.2)
- moved REF** 0.45 mm to (157.7, 123.2)
- moved S1 0.45 mm to (158.2, 128.8)
- moved C3 0.09 mm to (146.2, 125.1)
Routing:
- net PWR_GND: track 36.6 -> 204.9 mm
- net PWR_5V: track 90.4 -> 81.7 mm
- net Net-(J3-Pin_1): track 21.0 -> 15.8 mm
- net PWR_3V3: track 147.7 -> 152.4 mm
- net SDA: track 72.3 -> 76.6 mm
- net Net-(M1-D2): track 34.1 -> 30.1 mm
- net Net-(M1-D10): track 60.7 -> 57.4 mm
- net SCL: track 75.6 -> 73.5 mm
- net Net-(M1-D9): track 16.0 -> 17.6 mm
- net Net-(M1-D8): track 8.82 -> 9.34 mm
- added copper zone on F.Cu, net (none)
- removed copper zone on F.Cu, net PWR_GND
